File: schematic/analog_rev3/analog_rev3.kicad_sch (KiCad schematic)
At the start: 202 parts, among them J1 Jack, J10 Jack, J11 Jack, J12 Jack, J13 Jack, J14 Jack, J15 Jack, J16 Jack, J17 Jack, J18 Jack, J19 Jack, J2 Jack, J20 Jack, J21 Conn_01x07, J22 Conn_02x07, J23 Conn_02x07, J24 Conn_01x04, J25 Conn_01x04, J3 Jack, J4 Jack, J5 Jack, J6 Jack, J7 Jack, J8 Jack, J9 Jack, SW1 SW_Push, SW2 SW_Push, SW3 SW_Push, SW4 SW_Push, SW5 SW_Push, SW6 Encoder, SW7 Encoder, U1 LM339, U10 MCP6022, U11 LM833, U2 MCP6002, U3 MCP6002, U4 MCP6002, U5 MCP6002, U6 OPA2172, U7 OPA2172, U8 OPA2172, U9 OPA2172

Commit message: Minor fixes
Parts:
- J21: value Conn_01x07 -> OLED Display
- gave numbers to parts that had none: 2
Connections:
- net GND: now also C27.2, C28.1, C29.2, C30.1, C32.2, C33.1

Commit message: Update schematics, CC BY-SA with attribution to mxmxmx
Parts:
- C42, C43: value 8.2nF -> 8.2nF 5%
- C44, C45: value 1.0nF -> 1.0nF 5%
- J24, J25: value Conn_01x04 -> Trigger Inputs
- R100, R99: value 100K -> 100K 1%
- R101, R102: value 30.1K -> 31.6K 1%
- R93, R94: value 1.40K -> 1.40K 1%
- R95, R96: value 2.21K -> 2.21K 1%
- R97, R98: value 3.84K -> 3.84K 1%
- gave numbers to parts that had none: 4
Connections:
- net TR2: now reaches J22.13 (Pin_13), R24.2, R32.2, U1.13
- net DAC_E: now reaches J13.T, R79.2, R87.2
- net DAC_H: now reaches J16.T, R82.2, R90.2
- net TR4: now reaches J23.13 (Pin_13), R26.2, R34.2, U1.1
- net TR3: now reaches J23.14 (Pin_14), R25.2, R33.2, U1.2
- net TR1: now reaches J22.14 (Pin_14), R23.2, R31.2, U1.14
- net DAC_G: now reaches J15.T, R81.2, R89.2
- net DAC_F: now reaches J14.T, R80.2, R88.2
- net DAC_C: now reaches J11.T, R77.2, R85.2
- net DAC_D: now reaches J12.T, R78.2, R86.2
- net DAC_A: now reaches J9.T, R75.2, R83.2
- net DAC_B: now reaches J10.T, R76.2, R84.2
Other:
- company: (none) -> Copyright 2024 Paul Stoffregen, mxmxmx - CC BY-SA 4.0
- title: (none) -> O_C T4.1  Ornament and Crime optimized for Teensy 4.1
- moved on the sheet: C10, C12, C7, R11, R14, R16, R17, R20, R22, SW7

Commit message: converted gerbers to kicad_pcb files and added/customized footprints. generated new gerbers for testing and comparison.
still a few nuisance DRC warnings, mostly footprint quirks and silkscreen overlap, etc.

pcb files expect the included Custom_Footprints library to be added to the project
Parts:
- C1, C10, C11, C12, C13, C14, C15, C16, C17, C18, C19, C2, C20, C21, C22, C23, C24, C25, C26, C27, C28, C29, C3, C30, C31, C32, C33, C34, C35, C36, C37, C38, C39, C4, C40, C41, C42, C43, C44, C45, C46, C47, C48, C49, C5, C50, C51, C6, C7, C8, C9: footprint (none) -> Custom_Footprints:C_0805_2012Metric_Pad1.18x1.45mm_HandSolder_rectpads
- J1, J10, J11, J12, J13, J14, J15, J16, J17, J18, J19, J2, J20, J3, J4, J5, J6, J7, J8, J9: footprint (none) -> Custom_Footprints:Jack_3.5mm_QingPu_WQP-PJ398SM_Vertical_CircularHoles_reduced
- J21: footprint (none) -> Connector_PinHeader_2.54mm:PinHeader_1x07_P2.54mm_Vertical
- J22, J23: footprint (none) -> Custom_Footprints:PinHeader_2x07_P2.54mm_Vertical_reduced
- J24, J25: footprint (none) -> Custom_Footprints:PinHeader_1x04_P2.54mm_Vertical_reduced
- J26, J27: footprint (none) -> Custom_Footprints:PinHeader_1x16_P2.54mm_Vertical_reduced
- JP1, JP2, JP3, JP4: footprint (none) -> Jumper:SolderJumper-2_P1.3mm_Bridged_Pad1.0x1.5mm
- R1, R10, R100, R101, R102, R11, R12, R13, R14, R15, R16, R17, R18, R19, R2, R20, R21, R22, R23, R24, R25, R26, R27, R28, R29, R3, R30, R31, R32, R33, R34, R35, R36, R37, R38, R39, R4, R40, R41, R42, R43, R44, R45, R46, R47, R48, R49, R5, R50, R51, R52, R53, R54, R55, R56, R57, R58, R59, R6, R60, R61, R62, R63, R64, R65, R66, R67, R68, R69, R7, R70, R71, R72, R73, R74, R75, R76, R77, R78, R79, R8, R80, R81, R82, R83, R84, R85, R86, R87, R88, R89, R9, R90, R91, R92, R93, R94, R95, R96, R97, R98, R99: footprint (none) -> Custom_Footprints:R_0805_2012Metric_Pad1.20x1.40mm_HandSolder_rectpads
- SW1, SW2, SW3, SW4, SW5: footprint (none) -> Button_Switch_THT:SW_PUSH_6mm
- SW6, SW7: footprint (none) -> Custom_Footprints:RotaryEncoder_Alps_EC11E-Switch_Vertical_H20mm_CircularMountingHoles_s1s2-swap+roundA
- U1: footprint (none) -> Custom_Footprints:SOIC-14_3.9x8.7mm_P1.27mm_shiftedpads
- U10, U11, U2, U3, U4, U5, U6, U7, U8, U9: footprint (none) -> Custom_Footprints:SOIC-8_3.9x4.9mm_P1.27mm_shiftedpads

Commit message: added D6 per Paul's recommendation, to help protect U17
reduced pads on ADC footprint to help prevent solder bridging

updated a few footprint silkscreens to look more like original rev3 board

generated updated gerber zip files

TODO: update IC pads to match more closely to original rev3 board if it makes soldering easier
Parts:
- JP1, JP2, JP3, JP4: footprint Jumper:SolderJumper-2_P1.3mm_Bridged_Pad1.0x1.5mm -> Custom_Footprints:SolderJumper-2_P1.3mm_Bridged_Pad1.0x1.5mm_reduced
Changed lines of the file:
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@@
 			)
 		)
-		(property "Footprint" "Jumper:SolderJumper-2_P1.3mm_Bridged_Pad1.0x1.5mm"
+		(property "Footprint" "Custom_Footprints:SolderJumper-2_P1.3mm_Bridged_Pad1.0x1.5mm_reduced"
 			(at 125.73 166.37 0)
 			(effects
@@
 			)
 		)
-		(property "Footprint" "Jumper:SolderJumper-2_P1.3mm_Bridged_Pad1.0x1.5mm"
+		(property "Footprint" "Custom_Footprints:SolderJumper-2_P1.3mm_Bridged_Pad1.0x1.5mm_reduced"
 			(at 207.01 165.1 0)
 			(effects
@@
 			)
 		)
-		(property "Footprint" "Jumper:SolderJumper-2_P1.3mm_Bridged_Pad1.0x1.5mm"
+		(property "Footprint" "Custom_Footprints:SolderJumper-2_P1.3mm_Bridged_Pad1.0x1.5mm_reduced"
 			(at 43.18 166.37 0)
 			(effects
@@
 			)
 		)
-		(property "Footprint" "Jumper:SolderJumper-2_P1.3mm_Bridged_Pad1.0x1.5mm"
+		(property "Footprint" "Custom_Footprints:SolderJumper-2_P1.3mm_Bridged_Pad1.0x1.5mm_reduced"
 			(at 289.56 165.1 0)
 			(effects
